File: HW/piADAC/piADAC.kicad_pcb (KiCad board)
At the start: 2 copper layers, 64 x 55 mm, 75 parts, among them J1 Conn_2x20, J2 Conn_02x10_Odd_Even, J3 AudioJack2_Ground_Switch, J4 AudioJack2_Ground, J5 AudioJack2_Ground, J6 Conn_2x20, U1 PCM1863DBT, U2 AT24CS01-STUM, U3 ncp163, U4 ncp163, U5 ncp163, U6 PCM5242RHBR, X1 22.5792Mhz, X2 24.576Mhz

Commit message: finised ADAC hardware
Parts:
- removed R28, R7: 3K8, Resistor_SMD:R_0402_1005Metric
- added G***: LOGO, LOGO, F.Cu at (68.4, 43.6)
- added R26: 1.1kΩ, PCM_JLCPCB:R_0603, F.Cu at (57.8, 25.6)
- added R29: 2.7kΩ, PCM_JLCPCB:R_0603, F.Cu at (54.8, 25.6)
- added R30: 1.1kΩ, PCM_JLCPCB:R_0603, F.Cu at (42.0, 26.4)
- added R31: 2.7kΩ, PCM_JLCPCB:R_0603, F.Cu at (45.2, 26.4)
- added R32: 1.1kΩ, PCM_JLCPCB:R_0603, F.Cu at (45.2, 24.8)
- added R33: 2.7kΩ, PCM_JLCPCB:R_0603, F.Cu at (42.0, 24.8)
- D1, D2: footprint zynthiandac:led_0806 -> LED_THT:LED_D3.0mm
- R5: value 3K8 -> 1.1kΩ; footprint Resistor_SMD:R_0402_1005Metric -> PCM_JLCPCB:R_0603
- R6: value 3K8 -> 2.7kΩ; footprint Resistor_SMD:R_0402_1005Metric -> PCM_JLCPCB:R_0603
- moved D1 9.31 mm to (14.6, 28.2), turned to 90 degrees
- moved R5 4.95 mm to (57.8, 23.8), turned to 180 degrees
- moved D2 3.40 mm to (57.8, 37.6)
- moved R20 2.00 mm to (54.8, 39.0)
- moved R6 1.80 mm to (54.8, 23.8), turned to 180 degrees
Connections:
- J2 pad 15: Net-(J2-Pad15) -> unconnected-(J2-Pin_15-Pad15)
- J3 pad SN: Net-(J3-PadSN) -> unconnected-(J3-PadSN)
- J3 pad T: Net-(J3-PadT) -> unconnected-(J3-PadT)
- R5 pad 1: ID_SC -> DVDD
- R5 pad 2: DVDD -> Net-(R5-Pad2)
- R6 pad 1: ID_SD -> Net-(R5-Pad2)
- R6 pad 2: DVDD -> ID_SD
- U1 pad 10: Net-(U1-Pad10) -> unconnected-(U1-XI-Pad10)
- U1 pad 19: Net-(U1-Pad19) -> unconnected-(U1-GPIO3/INTC-Pad19)
- U1 pad 21: Net-(U1-Pad21) -> unconnected-(U1-GPIO1/INTA/DMIN-Pad21)
- U1 pad 27: Net-(U1-Pad27) -> unconnected-(U1-VINL4/VIN4M-Pad27)
- U1 pad 28: Net-(U1-Pad28) -> unconnected-(U1-VINR4/VIN3M-Pad28)
- U1 pad 29: Net-(U1-Pad29) -> unconnected-(U1-VINL3/VIN4P-Pad29)
- U1 pad 30: Net-(U1-Pad30) -> unconnected-(U1-VINR3/VIN3P-Pad30)
- U1 pad 9: Net-(U1-Pad9) -> unconnected-(U1-XO-Pad9)
- U3 pad 4: Net-(U3-Pad4) -> unconnected-(U3-NC-Pad4)
- U4 pad 4: Net-(U4-Pad4) -> unconnected-(U4-NC-Pad4)
- U5 pad 4: Net-(U5-Pad4) -> unconnected-(U5-NC-Pad4)
- U6 pad 19: Net-(U6-Pad19) -> unconnected-(U6-GPIO5-Pad19)
- U6 pad 29: Net-(U6-Pad29) -> unconnected-(U6-NC-Pad29)
- U6 pad 30: Net-(U6-Pad30) -> unconnected-(U6-NC-Pad30)
Routing:
- net Net-(D1-A): track 3.80 -> 15.5 mm
- net Net-(D1-K): track 1.52 -> 10.8 mm
- net Net-(D2-A): track 3.54 -> 12.0 mm
- net GND: track 692.6 -> 700.1 mm, vias 52 -> 54
- net DVDD: track 91.4 -> 97.3 mm, vias 6 -> 8
- net Net-(J1-p20): track 54.5 -> 56.4 mm
- net Net-(D2-K): track 1.65 -> 3.38 mm
- net Net-(J1-p21): track 34.0 -> 35.7 mm
- net Net-(J1-p19): track 49.4 -> 51.0 mm
- net Net-(R32-Pad2): track 0.00 -> 1.56 mm
- net Net-(R30-Pad2): track 0.00 -> 1.56 mm
- net Net-(U2-WP): track 3.68 -> 4.66 mm
- net ID_SC: track 17.0 -> 17.8 mm
- net ID_SD: track 10.9 -> 11.7 mm
Other:
- board text added: "15"
- board text added: "5V"
- board text added: "ESOF 423 Version 1"
- board text added: "gnd"
- board text added: "inl+"
- board text added: "inr+"
- board text added: "io14"
- board text added: "outl+"
- board text added: "outr+"
- board text added: "scl"
- board text added: "sda"
