File: HW/piADAC/piADAC.kicad_sch (KiCad schematic)
At the start: 75 parts, among them J1 Conn_2x20, J2 Conn_02x10_Odd_Even, J3 AudioJack2_Ground_Switch, J4 AudioJack2_Ground, J5 AudioJack2_Ground, J6 Conn_2x20, U1 PCM1863DBT, U2 AT24CS01-STUM, U3 ncp163, U4 ncp163, U5 ncp163, U6 PCM5242RHBR, X1 22.5792Mhz, X2 24.576Mhz

Commit message: finised ADAC hardware
Parts:
- removed R28, R5, R6, R7: 3K8, Resistor_SMD:R_0402_1005Metric, symbol Device:R
- added R26, R30, R32, R5: 1.1kΩ, PCM_JLCPCB:R_0603, symbol PCM_JLCPCB-Resistors:0603,1.1kΩ
- added R29, R31, R33, R6: 2.7kΩ, PCM_JLCPCB:R_0603, symbol PCM_JLCPCB-Resistors:0603,2.7kΩ
- D1, D2: footprint zynthiandac:led_0806 -> LED_THT:LED_D3.0mm
Connections:
- net DVDD: now also R26.1, R33.2, R5.1
- net GND: now also R30.1
- net ID_SC: now also R29.2
- net ID_SD: now also R6.2
- net at U2.5 (WP): now also R31.2, R32.1
- new net: R30.2, R31.1
- new net: R5.2, R6.1
- new net: R26.2, R29.1
- new net: R32.2, R33.1
Other:
- moved on the sheet: D2
